File: Hardware/Basic/smartwatch class 2.sch (EAGLE design)
At the start: 52 parts, among them SW3 SWITCH.MOM, SW4 SWITCH.MOM, SW5 SWITCH.MOM, U1 NRF52832_MODULE_MDBT42, U4 PCF8523

Commit message: finished class 2 video
Changed lines of the file:
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@@
 <text x="76.2" y="269.24" size="5.08" layer="91" font="vector" ratio="15">OLED</text>
 <text x="218.44" y="261.62" size="5.08" layer="91" font="vector" ratio="15">power management</text>
-<text x="157.48" y="297.18" size="5.08" layer="91" font="vector" ratio="15">buttons</text>
+<text x="154.94" y="287.02" size="5.08" layer="91" font="vector" ratio="15">buttons</text>
 <text x="-40.64" y="144.78" size="5.08" layer="91" font="vector" ratio="15">SD card</text>
 <text x="365.76" y="149.86" size="5.08" layer="91" font="vector" ratio="15">real-time clock</text>
 <text x="241.3" y="142.24" size="5.08" layer="91" font="vector" ratio="15">cortex debugger/programmer</text>
 <text x="287.02" y="96.52" size="5.08" layer="91" font="vector" ratio="15" rot="R180">RTC</text>
+<wire x1="-88.9" y1="307.34" x2="-81.28" y2="307.34" width="2.54" layer="94"/>
+<wire x1="-81.28" y1="307.34" x2="462.28" y2="307.34" width="2.54" layer="94"/>
+<wire x1="462.28" y1="307.34" x2="462.28" y2="-12.7" width="2.54" layer="94"/>
+<wire x1="462.28" y1="-12.7" x2="-91.44" y2="-12.7" width="2.54" layer="94"/>
+<wire x1="-91.44" y1="-12.7" x2="-91.44" y2="307.34" width="2.54" layer="94"/>
+<wire x1="-91.44" y1="309.88" x2="-91.44" y2="307.34" width="2.54" layer="94"/>
+<wire x1="-91.44" y1="307.34" x2="-88.9" y2="307.34" width="2.54" layer="94"/>
 </plain>
 <instances>

Commit message: deleted the second board and partially wired the board
Parts:
- removed C19: 2.2uF, LinnesLab-Passives:CAPACITOR0402
- removed C20, C21: 4.7u, LinnesLab-Passives:CAPACITOR0603
- removed CORTEX2: CORTEX_DEBUG_PTH, LinnesLab-Connectors:CORTEX_DEBUG_PTH
- removed D5: (no value), LinnesLab-DiscreteSemi:SCHOTTKY-USC
- removed R11: (no value), LinnesLab-Passives:RESISTOR0603
- removed R12, R13, R14, R15: 100k, LinnesLab-Passives:RESISTOR0603
- removed SD2: (no value), LinnesLab-Connectors:MICROSD
- removed U4: PCF8523, LinnesLab-Clocks:PCF8523
- removed USB2: USB.MICRO-BIGGERPADS, LinnesLab-Connectors:USB.MICRO-BIGGERPADS
- added C10, C9: (no value), LinnesLab-Passives:CAPACITOR0603
- added C7: 1u, LinnesLab-Passives:CAPACITOR0603
- added D3: (no value), LinnesLab-DiscreteSemi:SCHOTTKY-USC
- added DEBUG1: CORTEX_DEBUG_PTH, LinnesLab-Connectors:CORTEX_DEBUG_PTH
- added J1: FTDI_DEVICESMD, LinnesLab-Connectors:FTDI_DEVICESMD
- added R10: 10k, LinnesLab-Passives:RESISTOR0603
- added R3, R4: 1k, LinnesLab-Passives:RESISTOR0603
- added U2: NRF52832_MODULE_MDBT42, LinnesLab-Microcontrollers:NRF52832_MODULE_MDBT42
- C1: value 1u -> 10uF
- C11, C12: value 1u -> 300p
- C13: value 100n -> 4.7u
- C14, C15, C18: value 2.2uF -> 1u; device LinnesLab-Passives:CAPACITOR0402 -> LinnesLab-Passives:CAPACITOR0603
- C16: value 10uF -> 4.7u
- C17: value 2.2uF -> 100n; device LinnesLab-Passives:CAPACITOR0402 -> LinnesLab-Passives:CAPACITOR0603
- C2, C3: value (none) -> 2.2uF; device LinnesLab-Passives:CAPACITOR0603 -> LinnesLab-Passives:CAPACITOR0402
- C4, C5: value 300p -> 2.2uF; device LinnesLab-Passives:CAPACITOR0603 -> LinnesLab-Passives:CAPACITOR0402
- C6: value 10u -> 2.2uF; device LinnesLab-Passives:CAPACITOR0805 -> LinnesLab-Passives:CAPACITOR0402
- C8: value 1u -> 10u; device LinnesLab-Passives:CAPACITOR0603 -> LinnesLab-Passives:CAPACITOR0805
- R1: value 1k -> 10k
- R2: value 1k -> 390k
- R5, R8, R9: value 10k -> 100k
- R6: value 10k -> (none)
- R7: value 390k -> 100k
- SW2: value (none) -> SWITCH.MOM; device LinnesLab-Switches:SPST-PTS830GG140-COPY.1-3 -> LinnesLab-Switches:SWITCH.MOM
- SW5: value SWITCH.MOM -> (none); device LinnesLab-Switches:SWITCH.MOM -> LinnesLab-Switches:SPST-PTS830GG140-COPY.1-3
- U1: value NRF52832_MODULE_MDBT42 -> (none); device LinnesLab-Microcontrollers:NRF52832_MODULE_MDBT42 -> LinnesLab-Displays:DISP_OLED_UG-2864HSWEG01-NO-WRAPAROUND
- U3: value (none) -> PCF8523; device LinnesLab-Displays:DISP_OLED_UG-2864HSWEG01-NO-WRAPAROUND -> LinnesLab-Clocks:PCF8523; DIGIKEY (none) -> 568-5306-1-ND; I2C_ADDRESS (none) -> 0x68h; MFN (none) -> PCF8523T/1,118; MFN_MANUFACTURER (none) -> NXP USA Inc.
- renumbered CHRG2 to CHRG1, D4 to D1, LDO2 to LDO1, XTAL3 to XTAL2
Connections:
- removed net BATT: R13.1, R14.2
- removed net CD1: SD2.CARD_DETECT
- removed net CD2: SD2.CARD_DETECT1
- removed net CHRG.STAT: CHRG1.STAT, R12.1
- removed net CS.OLED: U3./CS
- removed net DC.OLED: U3.DC/I2C_SA0
- removed net RESET.OLED: U3./RES
- removed net SD.CS: SD2.CS
- removed net USB+: USB2.D+
- removed net USB-: USB2.D-
- new net A4/PPG: U2.P0.28/AIN4
- new net A5/TIA: U2.P0.29/AIN5
- new net A7.BATT: R8.1, R9.2
- new net A7/BATT: U2.P0.31/AIN7
- new net D11/SW1: SW2.1, U2.P0.11
- new net D15/SW2: SW3.1, U2.P0.15
- new net D16/CS.OLED: U1./CS, U2.P0.16
- new net D27/CHRG.STAT: CHRG1.STAT, R5.1
- new net D27/CHRG.STATUS: U2.P0.27
- new net D3/RESET.OLED: U1./RES, U2.P0.03/AIN1
- new net D30/LED.CTRL: U2.P0.30/AIN6
- new net D4/DC.OLED: U1.DC/I2C_SA0, U2.P0.04/AIN2
- new net D5/CD1: U2.P0.05/AIN3
- new net D7/SD.CS: U2.P0.07
- new net RXD.NRF: J1.TXO
- new net TXD.NRF: J1.RXI
- net 3.3V: now also C15.1, C18.1, C5.2, C8.2, D3.C, DEBUG1.VCC, R10.2, R7.2, U1.VBAT, U2.VDD; no longer C12.1, C17.2, C19.2, C8.1, CORTEX2.VCC, D2.C, R15.2, R6.2, R8.2, R9.2, SD2.VDD, U3.VBAT, U4.VDD
- net DFU: now also U2.P0.20; no longer U1.P0.20
- net DTR: now also C17.1, J1.DTR; no longer C13.1
- net FRST: now also U2.P0.22; no longer U1.P0.22
- net GND: now also C1.1, C10.2, C11.2, C13.1, C14.1, C15.2, C16.2, C18.2, C3.1, C5.1, C7.2, C8.1, C9.1, DEBUG1.GND@3, DEBUG1.GND@5, DEBUG1.GNDDTCT, DEBUG1.KEY, J1.CTS, J1.GND, R1.1, R2.2, R6.1, R7.1, R9.1, SW2.3, SW3.3, SW5.B, U1.BS0, U1.BS2, U1.NC(GND)@1, U1.NC(GND)@2, U1.VLSS, U1.VSS, U2.GND@1, U2.GND@2, U2.GND@3, U2.GND@4; no longer C1.2, C11.1, C16.1, C17.1, C18.1, C19.1, C2.1, C20.2, C21.1, C3.2, C4.2, C5.2, C8.2, CORTEX2.GND@3, CORTEX2.GND@5, CORTEX2.GNDDTCT, CORTEX2.KEY, R11.1, R14.1, R15.1, R5.1, R7.2, SD2.GND, SD2.GND1, SD2.VSS, SW2.B, U1.GND@1, U1.GND@2, U1.GND@3, U1.GND@4, U3.BS0, U3.BS2, U3.NC(GND)@1, U3.NC(GND)@2, U3.VLSS, U4.VSS, USB2.GND
- net LED1: now also R3.2, U2.P0.17; no longer R1.2, U1.P0.17
- net LED2: now also R4.2, U2.P0.19; no longer R2.2, U1.P0.19
- net MISO: now also U2.P0.14; no longer SD2.DATA_OUT, U1.P0.14
- net MOSI: now also U1.D1/SPI_SDIN/I2C_SDA, U2.P0.13; no longer SD2.DATA_IN, U1.P0.13, U3.D1/SPI_SDIN/I2C_SDA
- net N$1: now also C9.2, U2.P0.00/XL1; no longer C2.2, U1.P0.00/XL1
- net N$10: now also C4.1, U1.C2N; no longer C14.1, U3.C2N
- net N$11: now also C2.2, U1.C1P; no longer C15.2, U3.C1P
- net N$12: now also C2.1, U1.C1N; no longer C15.1, U3.C1N
- net N$13: now also DEBUG1.NC/TDI; no longer CORTEX2.NC/TDI
- net N$14: now also C1.2, U1.VCC; no longer C16.2, U3.VCC
- net N$15: now also C3.2, U1.VCOMH; no longer C18.2, U3.VCOMH
- net N$17: now also R6.2; no longer R11.2
- net N$19: now also U3.OSCO; no longer U4.OSCO
- net N$2: now also C10.1, U2.P0.01/XL2; no longer C3.1, U1.P0.01/XL2
- net N$20: now also U3.OSCI; no longer U4.OSCI
- net N$3: now also U2.DCC; no longer U1.DCC
- net N$4: now also R1.2, U1.BS1; no longer R5.2, U3.BS1
- net N$5: now also R3.1; no longer R1.1
- net N$6: now also R2.1, U1.IREF; no longer R7.1, U3.IREF
- net N$7: now also R4.1; no longer R2.1
- net N$8: now also C7.1, U2.DEC4; no longer C1.1, U1.DEC4
- net N$9: now also C4.2, U1.C2P; no longer C14.2, U3.C2P
- net P0.09/NFC1: now also C11.1, U2.P0.09; no longer C5.1, U1.P0.09
- net P0.10/NFC2: now also C12.1, U2.P0.10; no longer C4.1, U1.P0.10
- net RESET: now also C17.2, D3.A, DEBUG1.!RESET, R10.1, SW5.A, U2.P0.21/RESET; no longer C13.2, CORTEX2.!RESET, D2.A, R6.1, SW2.A, U1.P0.21/RESET
- net RXD: now also U2.P0.08; no longer U1.P0.08
- net SCK: now also U1.D0/SPI_SCLK/I2C_SCK, U2.P0.12; no longer SD2.SCLK, U1.P0.12, U3.D0/SPI_SCLK/I2C_SCK
- net SCL: now also U2.P0.26, U3.SCL; no longer R8.1, U1.P0.26, U4.SCL
- net SDA: now also U2.P0.25, U3.SDA; no longer R9.1, U1.P0.25, U4.SDA
- net SWCLK: now also DEBUG1.SWDCLK/TCK, U2.SWDCLK; no longer CORTEX2.SWDCLK/TCK, U1.SWDCLK
- net SWDIO: now also DEBUG1.SWDIO/TMS, U2.SWDIO; no longer CORTEX2.SWDIO/TMS, U1.SWDIO
- net SWO: now also DEBUG1.SWO/TDO, U2.P0.18/SWO; no longer CORTEX2.SWO/TDO, U1.P0.18/SWO
- net TXD: now also U2.P0.06; no longer U1.P0.06
- net VBATT: now also U3.VBAT; no longer U4.VBAT
- net VIN: now also C13.2, C14.2, D2.C, R5.2; no longer C11.2, C21.2, D5.C, R12.2
- net VLIPO: now also C16.1, R8.2; no longer C20.1, R13.2
- net V_USB: now also D2.A, J1.VCC; no longer D5.A, USB2.V+
Other:
- note removed: "Connect MISO, MOSI, and SCK to appropriate pins on microcontroller. Those are SPI pins and are generally prespecified. You have more flexibility with the SD.CS pin."
- note removed: "SD card"
- moved on the sheet: C1, C11, C12, C13, C14, C15, C16, C17, C18, C2, C3, C4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
