File: Hardware/Basic/smartwatch class 2_justincase.brd (EAGLE design)
At the start: 38 x 38 mm, 49 parts, among them J1 FTDI_DEVICESMD, SW2 SWITCH.MOM, SW3 SWITCH.MOM, SW4 SWITCH.MOM, U2 NRF52832_MODULE_MDBT42, U3 PCF8523

Commit message: at 14:14 of video 2
Parts:
- C2, C3, C4, C5, C6: device LinnesLab-Passives:C0402 -> LinnesLab-Passives:C0603
- moved LDO1 15.5 mm to (2.97, 4.42), turned to 180 degrees
- moved C18 13.7 mm to (2.54, 1.80)
- moved R9 13.5 mm to (-3.81, 4.80)
- moved R8 9.91 mm to (-1.83, 4.88)
- moved C16 9.73 mm to (6.91, 13.1), turned to 180 degrees
- moved D1 9.58 mm to (1.45, 9.93), turned to 270 degrees
- moved C14 9.35 mm to (2.46, 7.24), turned to 0 degrees
- moved D2 5.79 mm to (3.12, 9.88), turned to 270 degrees
- moved R5 5.19 mm to (7.62, 3.53)
- moved CHRG1 4.93 mm to (7.67, 7.87), turned to 90 degrees
- moved C13 4.76 mm to (5.13, 7.87)
- moved C5 4.60 mm to (12.0, 22.3)
- moved C10 3.58 mm to (14.7, 22.3), turned to 90 degrees
- moved R6 3.30 mm to (7.37, 5.28), turned to 180 degrees
- moved C2 2.29 mm to (10.4, 22.3), turned to 270 degrees
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Connections:
- removed net RXD: U2.21
- removed net TXD: U2.19
- net RXD.NRF: now also U2.21
- net TXD.NRF: now also U2.19
Routing:
- net TXD.NRF: track 0.00 -> 24.4 mm, vias 0 -> 1
- net GND: track 27.9 -> 51.3 mm, vias 3 -> 8
- net RXD.NRF: track 0.00 -> 19.9 mm, vias 0 -> 1
- net VIN: track 0.00 -> 18.1 mm
- net VLIPO: track 0.00 -> 13.6 mm
- net V_USB: track 0.00 -> 11.2 mm, vias 0 -> 1
- net N$8: track 5.19 -> 0.25 mm
- net D27/CHRG.STAT: track 0.00 -> 3.60 mm
- net N$3: track 3.01 -> 0.00 mm
- net N$10: track 3.47 -> 6.06 mm
- net N$12: track 3.87 -> 6.03 mm
- net N$1: track 5.12 -> 6.97 mm
- net N$17: track 0.00 -> 1.70 mm
- net N$2: track 7.64 -> 9.12 mm
- net N$11: track 3.62 -> 4.46 mm
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
Commit message: video 2 35:46 but may be all wired up anyway
Parts:
- moved C17 19.9 mm to (35.5, 8.38)
- moved R9 17.0 mm to (4.45, 19.7), turned to 90 degrees
- moved R8 15.1 mm to (1.65, 19.6)
- moved R10 15.0 mm to (35.6, 13.4), turned to 180 degrees
- moved D3 11.3 mm to (35.4, 11.1), turned to 180 degrees
- moved R2 7.69 mm to (25.8, 13.0), turned to 180 degrees
- moved R1 6.15 mm to (17.0, 13.1), turned to 180 degrees
- moved SW5 3.15 mm to (31.9, 11.6), turned to 270 degrees
- moved C15 2.12 mm to (1.50, 25.6)
- moved L1 1.44 mm to (15.4, 26.6), turned to 0 degrees
- moved C4 0.89 mm to (8.00, 22.2)
- moved C7 0.67 mm to (15.3, 28.0)
- moved C2 0.66 mm to (9.78, 22.3)
- moved XTAL1 0.54 mm to (18.5, 21.7)
- moved C6 0.51 mm to (12.9, 22.3)
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Routing:
- net GND: track 51.3 -> 107.3 mm, vias 8 -> 15
- net D15/SW2: track 0.00 -> 26.9 mm, vias 0 -> 2
- net DTR: track 0.00 -> 26.5 mm, vias 0 -> 1
- net D11/SW1: track 0.00 -> 26.3 mm, vias 0 -> 2
- net D16/CS.OLED: track 0.00 -> 16.7 mm, vias 0 -> 2
- net MOSI: track 0.00 -> 15.3 mm, vias 0 -> 2
- net SCK: track 0.00 -> 12.0 mm, vias 0 -> 2
- net VLIPO: track 13.6 -> 25.2 mm
- net N$8: track 0.25 -> 11.8 mm
- net RESET: track 9.58 -> 19.1 mm
- net D4/DC.OLED: track 0.00 -> 7.48 mm
- net D3/RESET.OLED: track 0.00 -> 7.48 mm
- net N$3: track 0.00 -> 6.29 mm
- net N$6: track 0.00 -> 4.78 mm
- net N$4: track 0.00 -> 4.65 mm
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
Commit message: just hooked up the A7.batt
Parts:
- moved C15 0.26 mm to (1.75, 25.5)
Connections:
- removed net A7/BATT: U2.8
- net A7.BATT: now also U2.8
Routing:
- net A7.BATT: track 2.84 -> 25.6 mm
- net GND: track 107.3 -> 113.4 mm, vias 15 -> 16
Changed lines of the file:
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@@
 <attribute name="NAME" x="1.8288" y="7.874" size="0.6604" layer="25"/>
 </element>
-<element name="C15" library="LinnesLab-Passives" package="C0603" package3d_urn="urn:adsk.eagle:package:15661989/2" value="1u" x="1.4986" y="25.5524" smashed="yes" rot="R90">
-<attribute name="NAME" x="1.9558" y="27.3558" size="0.6604" layer="25" rot="R90"/>
+<element name="C15" library="LinnesLab-Passives" package="C0603" package3d_urn="urn:adsk.eagle:package:15661989/2" value="1u" x="1.7526" y="25.527" smashed="yes" rot="R90">
+<attribute name="NAME" x="2.2098" y="27.3304" size="0.6604" layer="25" rot="R90"/>
 </element>
 <element name="C16" library="LinnesLab-Passives" package="C0603" package3d_urn="urn:adsk.eagle:package:15661989/2" value="4.7u" x="6.9088" y="13.081" smashed="yes" rot="R180">
@@
 <wire x1="36.7284" y1="18.69" x2="36.6058" y2="18.5674" width="0.1524" layer="1"/>
 <via x="36.6058" y="18.5674" extent="1-16" drill="0.35"/>
-<via x="30.3276" y="32.5374" extent="1-16" drill="0.35"/>
+<via x="31.2166" y="32.7914" extent="1-16" drill="0.35"/>
 <wire x1="29.1872" y1="33.1624" x2="29.1872" y2="33.1176875" width="0.1524" layer="1"/>
-<wire x1="29.7674875" y1="32.5374" x2="29.1872" y2="33.1176875" width="0.1524" layer="1"/>
-<wire x1="29.7674875" y1="32.5374" x2="30.3276" y2="32.5374" width="0.1524" layer="1"/>
+<wire x1="29.5134875" y1="32.7914" x2="29.1872" y2="33.1176875" width="0.1524" layer="1"/>
+<wire x1="29.5134875" y1="32.7914" x2="31.2166" y2="32.7914" width="0.1524" layer="1"/>
 <wire x1="35.3058" y1="34.2524" x2="34.5306" y2="33.4772" width="0.1524" layer="1"/>
 <wire x1="34.5306" y1="33.4772" x2="34.00589375" y2="33.4772" width="0.1524" layer="1"/>
-<wire x1="33.06609375" y1="32.5374" x2="30.3276" y2="32.5374" width="0.1524" layer="1"/>
-<wire x1="34.00589375" y1="33.4772" x2="33.06609375" y2="32.5374" width="0.1524" layer="1"/>
+<wire x1="32.73589375" y1="32.2072" x2="31.8008" y2="32.2072" width="0.1524" layer="1"/>
+<wire x1="31.8008" y1="32.2072" x2="31.2166" y2="32.7914" width="0.1524" layer="1"/>
+<wire x1="34.00589375" y1="33.4772" x2="32.73589375" y2="32.2072" width="0.1524" layer="1"/>
 <wire x1="19.9872" y1="33.1624" x2="20.5106" y2="32.639" width="0.1524" layer="1"/>
 <wire x1="20.5106" y1="32.639" x2="22.4282" y2="32.639" width="0.1524" layer="1"/>
@@
 <wire x1="18.123" y1="6.7966" x2="18.123" y2="6.0834" width="0.1524" layer="1"/>
 <wire x1="18.123" y1="6.0834" x2="15.748" y2="3.7084" width="0.1524" layer="1"/>
+<wire x1="3.7" y1="27.6098" x2="2.4672" y2="26.377" width="0.1524" layer="1"/>
+<wire x1="2.4672" y1="26.377" x2="1.7526" y2="26.377" width="0.1524" layer="1"/>
+<wire x1="3.8608" y1="24.3704" x2="2.4672" y2="25.764" width="0.1524" layer="1"/>
+<wire x1="2.4672" y1="25.764" x2="2.4672" y2="26.377" width="0.1524" layer="1"/>
+<wire x1="2.4672" y1="26.377" x2="2.8346" y2="26.0096" width="0.1524" layer="1"/>
+<wire x1="2.8346" y1="26.0096" x2="3.1496" y2="26.0096" width="0.1524" layer="1"/>
+<via x="3.1496" y="26.0096" extent="1-16" drill="0.35"/>
 <wire x1="35.814" y1="31.9786" x2="35.814" y2="30.7086" width="0" layer="19" extent="1-1"/>
 <wire x1="35.814" y1="29.4386" x2="35.814" y2="30.7086" width="0" layer="19" extent="1-1"/>
@@
 <wire x1="2.9718" y1="5.7197" x2="5.1308" y2="7.024" width="0" layer="19" extent="1-1"/>
 <wire x1="12.7254" y1="4.826" x2="8.216" y2="5.2832" width="0" layer="19" extent="1-16"/>
-<wire x1="3.8608" y1="24.3704" x2="4.445" y2="18.8096" width="0" layer="19" extent="1-1"/>
-<wire x1="1.4986" y1="26.4024" x2="3.8608" y2="24.3704" width="0" layer="19" extent="1-1"/>
-<wire x1="3.7" y1="27.6098" x2="1.4986" y2="26.4024" width="0" layer="19" extent="1-1"/>
+<wire x1="3.1496" y1="26.0096" x2="4.445" y2="18.8096" width="0" layer="19" extent="1-1"/>
 </signal>
 <signal name="SWDIO">
@@
 <contactref element="U2" pad="36"/>
 <contactref element="DEBUG1" pad="4"/>
-<wire x1="29.1872" y1="30.8624" x2="29.43614375" y2="30.8624" width="0.1524" layer="1"/>
-<wire x1="29.43614375" y1="30.8624" x2="32.193971875" y2="28.104571875" width="0.1524" layer="1"/>
-<wire x1="32.193971875" y1="28.104571875" x2="34.479971875" y2="28.104571875" width="0.1524" layer="1"/>
+<wire x1="29.1872" y1="30.8624" x2="29.84254375" y2="30.8624" width="0.1524" layer="1"/>
+<wire x1="29.84254375" y1="30.8624" x2="32.600371875" y2="28.104571875" width="0.1524" layer="1"/>
+<wire x1="32.600371875" y1="28.104571875" x2="34.479971875" y2="28.104571875" width="0.1524" layer="1"/>
 <wire x1="34.479971875" y1="28.104571875" x2="34.544" y2="28.1686" width="0.1524" layer="1"/>
 </signal>
@@
 <contactref element="DEBUG1" pad="10"/>
 <via x="32.07779375" y="27.4388" extent="1-16" drill="0.35"/>
-<wire x1="32.07779375" y1="27.4388" x2="32.0660875" y2="27.4388" width="0.1524" layer="1"/>
-<wire x1="32.0660875" y1="27.4388" x2="29.3424875" y2="30.1624" width="0.1524" layer="1"/>
-<wire x1="29.1872" y1="30.1624" x2="29.3424875" y2="30.1624" width="0.1524" layer="1"/>
+<wire x1="32.07779375" y1="27.4388" x2="32.07779375" y2="27.98589375" width="0.1524" layer="1"/>
+<wire x1="32.07779375" y1="27.98589375" x2="29.9012875" y2="30.1624" width="0.1524" layer="1"/>
+<wire x1="29.1872" y1="30.1624" x2="29.9012875" y2="30.1624" width="0.1524" layer="1"/>
 <wire x1="32.07779375" y1="27.4388" x2="32.07779375" y2="29.51239375" width="0.1524" layer="16"/>
 <wire x1="32.07779375" y1="29.51239375" x2="34.544" y2="31.9786" width="0.1524" layer="16"/>
@@
 <contactref element="R3" pad="2"/>
 <contactref element="U2" pad="31"/>
-<wire x1="29.1872" y1="27.3624" x2="29.5844" y2="27.3624" width="0.1524" layer="1"/>
-<wire x1="32.3224" y1="24.6244" x2="34.798" y2="24.6244" width="0.1524" layer="1"/>
-<wire x1="29.5844" y1="27.3624" x2="32.3224" y2="24.6244" width="0.1524" layer="1"/>
+<wire x1="29.1872" y1="27.3624" x2="30.0162" y2="27.3624" width="0.1524" layer="1"/>
+<wire x1="32.7542" y1="24.6244" x2="34.798" y2="24.6244" width="0.1524" layer="1"/>
+<wire x1="30.0162" y1="27.3624" x2="32.7542" y2="24.6244" width="0.1524" layer="1"/>
 </signal>
 <signal name="LED2">
@@
 <wire x1="1.651" y1="20.408" x2="1.7526" y2="20.5096" width="0.1524" layer="1"/>
 <wire x1="1.7526" y1="20.5096" x2="4.445" y2="20.5096" width="0.1524" layer="1"/>
+<contactref element="U2" pad="8"/>
+<wire x1="4.445" y1="20.5096" x2="7.2724" y2="23.337" width="0.1524" layer="1"/>
+<wire x1="7.2724" y1="23.337" x2="7.2724" y2="23.6688875" width="0.1524" layer="1"/>
+<wire x1="20.8818875" y1="23.3938" x2="21.0158" y2="23.5277125" width="0.1524" layer="1"/>
+<wire x1="21.0158" y1="25.5970875" x2="20.8818875" y2="25.731" width="0.1524" layer="1"/>
+<wire x1="21.0158" y1="23.5277125" x2="21.0158" y2="25.5970875" width="0.1524" layer="1"/>
+<wire x1="20.8818875" y1="25.731" x2="20.2186" y2="25.731" width="0.1524" layer="1"/>
+<wire x1="20.2186" y1="25.731" x2="19.9872" y2="25.9624" width="0.1524" layer="1"/>
+<wire x1="17.1317375" y1="23.3938" x2="20.8818875" y2="23.3938" width="0.1524" layer="1"/>
+<wire x1="7.2724" y1="23.6688875" x2="8.7975125" y2="25.194" width="0.1524" layer="1"/>
+<wire x1="8.7975125" y1="25.194" x2="15.3315375" y2="25.194" width="0.1524" layer="1"/>
+<wire x1="15.3315375" y1="25.194" x2="17.1317375" y2="23.3938" width="0.1524" layer="1"/>
 </signal>
 <signal name="VIN">
@@
 <contactref element="U2" pad="7"/>
 </signal>
-<signal name="A7/BATT">
-<contactref element="U2" pad="8"/>
-</signal>
 <signal name="D16/CS.OLED">
