File: Hardware/Basic/smartwatch class 2_justincase.sch (EAGLE design)
At the start: 49 parts, among them J1 FTDI_DEVICESMD, SW2 SWITCH.MOM, SW3 SWITCH.MOM, SW4 SWITCH.MOM, U2 NRF52832_MODULE_MDBT42, U3 PCF8523

Commit message: at 14:14 of video 2
Parts:
- C2, C3, C4, C5, C6: device LinnesLab-Passives:CAPACITOR0402 -> LinnesLab-Passives:CAPACITOR0603
Connections:
- removed net RXD: U2.P0.08
- removed net TXD: U2.P0.06
- net RXD.NRF: now also U2.P0.08
- net TXD.NRF: now also U2.P0.06
Changed lines of the file:
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@@
 <part name="LED2" library="LinnesLab-LED" deviceset="LED" device="0603" package3d_urn="urn:adsk.eagle:package:18593052/2" value="BLUE"/>
 <part name="GND20" library="LinnesLab-Symbols" deviceset="GND" device=""/>
-<part name="C4" library="LinnesLab-Passives" deviceset="CAPACITOR" device="0402" package3d_urn="urn:adsk.eagle:package:15402268/2" value="2.2uF"/>
-<part name="C2" library="LinnesLab-Passives" deviceset="CAPACITOR" device="0402" package3d_urn="urn:adsk.eagle:package:15402268/2" value="2.2uF"/>
+<part name="C4" library="LinnesLab-Passives" deviceset="CAPACITOR" device="0603" package3d_urn="urn:adsk.eagle:package:15661989/2" value="2.2uF"/>
+<part name="C2" library="LinnesLab-Passives" deviceset="CAPACITOR" device="0603" package3d_urn="urn:adsk.eagle:package:15661989/2" value="2.2uF"/>
 <part name="C1" library="LinnesLab-Passives" deviceset="CAPACITOR" device="0603" package3d_urn="urn:adsk.eagle:package:15661989/2" value="10uF"/>
-<part name="C6" library="LinnesLab-Passives" deviceset="CAPACITOR" device="0402" package3d_urn="urn:adsk.eagle:package:15402268/2" value="2.2uF"/>
-<part name="C3" library="LinnesLab-Passives" deviceset="CAPACITOR" device="0402" package3d_urn="urn:adsk.eagle:package:15402268/2" value="2.2uF"/>
-<part name="C5" library="LinnesLab-Passives" deviceset="CAPACITOR" device="0402" package3d_urn="urn:adsk.eagle:package:15402268/2" value="2.2uF"/>
+<part name="C6" library="LinnesLab-Passives" deviceset="CAPACITOR" device="0603" package3d_urn="urn:adsk.eagle:package:15661989/2" value="2.2uF"/>
+<part name="C3" library="LinnesLab-Passives" deviceset="CAPACITOR" device="0603" package3d_urn="urn:adsk.eagle:package:15661989/2" value="2.2uF"/>
+<part name="C5" library="LinnesLab-Passives" deviceset="CAPACITOR" device="0603" package3d_urn="urn:adsk.eagle:package:15661989/2" value="2.2uF"/>
 <part name="U1" library="LinnesLab-Displays" deviceset="DISP_OLED_UG-2864HSWEG01" device="-NO-WRAPAROUND"/>
 <part name="GND21" library="LinnesLab-Symbols" deviceset="GND" device=""/>
@@
 </segment>
 </net>
-<net name="RXD" class="0">
-<segment>
-<wire x1="116.84" y1="66.04" x2="116.84" y2="68.58" width="0.1524" layer="91"/>
-<pinref part="U2" gate="G$1" pin="P0.08"/>
-<label x="116.84" y="66.04" size="1.27" layer="95" rot="R270" xref="yes"/>
-</segment>
-</net>
-<net name="TXD" class="0">
-<segment>
-<wire x1="111.76" y1="66.04" x2="111.76" y2="68.58" width="0.1524" layer="91"/>
-<pinref part="U2" gate="G$1" pin="P0.06"/>
-<label x="111.76" y="66.04" size="1.27" layer="95" rot="R270" xref="yes"/>
-</segment>
-</net>
 <net name="DTR" class="0">
 <segment>
@@
 <label x="162.56" y="190.5" size="1.778" layer="95"/>
 </segment>
+<segment>
+<wire x1="116.84" y1="66.04" x2="116.84" y2="68.58" width="0.1524" layer="91"/>
+<pinref part="U2" gate="G$1" pin="P0.08"/>
+<label x="116.84" y="66.04" size="1.27" layer="95" rot="R270" xref="yes"/>
+</segment>
 </net>
 <net name="TXD.NRF" class="0">
@@
 <label x="162.56" y="193.04" size="1.778" layer="95"/>
 </segment>
-</net>
+<segment>
+<wire x1="111.76" y1="66.04" x2="111.76" y2="68.58" width="0.1524" layer="91"/>
+<pinref part="U2" gate="G$1" pin="P0.06"/>
+<label x="111.76" y="66.04" size="1.27" layer="95" rot="R270" xref="yes"/>
+</segment>
+</net>

Commit message: just hooked up the A7.batt
Connections:
- removed net A7/BATT: U2.P0.31/AIN7
- net A7.BATT: now also U2.P0.31/AIN7
Changed lines of the file:
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@@
 <label x="292.1" y="220.98" size="1.27" layer="95" xref="yes"/>
+</segment>
+<segment>
+<pinref part="U2" gate="G$1" pin="P0.31/AIN7"/>
+<wire x1="86.36" y1="91.44" x2="83.82" y2="91.44" width="0.1524" layer="91"/>
+<label x="83.82" y="91.44" size="1.27" layer="95" rot="R180" xref="yes"/>
 </segment>
 </net>
@@
 </segment>
 </net>
-<net name="A7/BATT" class="0">
-<segment>
-<pinref part="U2" gate="G$1" pin="P0.31/AIN7"/>
-<wire x1="86.36" y1="91.44" x2="83.82" y2="91.44" width="0.1524" layer="91"/>
-<label x="83.82" y="91.44" size="1.27" layer="95" rot="R180" xref="yes"/>
-</segment>
-</net>
